File: crossometer-mini.kicad_sch (KiCad schematic)
At the start: 63 parts, among them J1 UART, J2 BAT, J3 AUX, J4 I²C, J5 USB_C_Receptacle_USB2.0, J6 Micro_SD_Card_Det, Q1 2N7002, Q2 CJ2301, Q3 UMH3N, SW1 IO0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

Commit message: add LCSC field to schematic
Parts:
- C1, C10, C7, C9: LCSC (none) -> C52923
- C11, C13, C14, C2, C3, C4, C5, C6, C8: LCSC (none) -> C1525
- C12: LCSC (none) -> C15525
- D1: LCSC (none) -> C965790
- D2: LCSC (none) -> C8598
- J5: LCSC (none) -> C319148
- J6: LCSC (none) -> C585350
- Q1: LCSC (none) -> C8545
- Q2: LCSC (none) -> C2910170
- Q3: LCSC (none) -> C62892
- R1, R5: LCSC (none) -> C4109
- R10, R14, R15, R16, R17, R2, R3, R4, R6, R7, R8, R9: LCSC (none) -> C25744
- R11, R12, R13, R18, R19, R20, R21, R22, R23: LCSC (none) -> C25741
- SW1, SW3: LCSC (none) -> C115357
- SW2: LCSC (none) -> C221841
- U1: LCSC (none) -> C83291
- U2: LCSC (none) -> C32574
- U3: LCSC (none) -> C967633
- U4: LCSC (none) -> C82899
- U5: LCSC (none) -> C82942
- U6: LCSC (none) -> C84681
